Commit message: Fix RViz topics, integrate Depth Anything V2 neural model, and fix geometric traversability projection

File: src/ugv_description/urdf/sensors/camera.urdf.xacro (robot description, xacro)
@@ -24,15 +24,23 @@
         </inertial>
     </link>
+    <!-- Tugbot camera_front link matching Gazebo SDF pose (0.0553, 0, 0.4323) -->
     <joint name="base_camera_joint" type="fixed">
         <parent link="base_link" />
         <child link="camera_link" />
-        <origin xyz="${base_length / 2.0 + camera_length / 2.0} 0 ${base_height / 2.0 + 0.05}" rpy="0 0 0" />
+        <origin xyz="0.0553 0 0.4323" rpy="0 0 0" />
     </joint>
-    <!-- Standard ROS optical frame convention (X forward -> Z forward, Y left -> -X left, Z up -> -Y down) -->
+    <!-- Standard ROS optical frame convention -->
     <link name="camera_link_optical" />
     <joint name="camera_optical_joint" type="fixed">
-        <origin xyz="0 0 0" rpy="${-pi/2} 0 ${-pi/2}" />
+        <origin xyz="0 0.0325 0.0125" rpy="${-pi/2} 0 ${-pi/2}" />
         <parent link="camera_link" />
         <child link="camera_link_optical" />
+    </joint>
+    <!-- Alias for Gazebo Tugbot frame_id: tugbot/camera_front/color -->
+    <link name="tugbot/camera_front/color" />
+    <joint name="tugbot_camera_color_joint" type="fixed">
+        <origin xyz="0 0 0" rpy="0 0 0" />
+        <parent link="camera_link_optical" />
+        <child link="tugbot/camera_front/color" />
     </joint>
     <gazebo reference="camera_link">

File: src/ugv_description/urdf/ugv_base.urdf.xacro (robot description, xacro)
@@ -11,10 +11,8 @@
     <link name="base_link">
         <visual>
+            <origin xyz="0 0 0" rpy="0 0 0" />
             <geometry>
-                <box size="${base_length} ${base_width} ${base_height}" />
+                <mesh filename="package://ugv_description/meshes/base/tugbot_simp.dae" />
             </geometry>
-            <material name="blue">
-                <color rgba="0.1 0.3 0.8 1.0" />
-            </material>
         </visual>
         <collision>
@@ -40,10 +38,8 @@
         <link name="${prefix}_wheel_link">
             <visual>
+                <origin xyz="0 0 0" rpy="0 0 0" />
                 <geometry>
-                    <cylinder radius="${wheel_radius}" length="${wheel_length}" />
+                    <mesh filename="package://ugv_description/meshes/wheel/wheel.dae" />
                 </geometry>
-                <material name="black">
-                    <color rgba="0.05 0.05 0.05 1.0" />
-                </material>
             </visual>
             <collision>

Commit message: feat: create Localbot — project-native robot replacing Fuel TugBot dependency
## Localbot: Custom Robot Model (src/ugv_sim/models/localbot/)

Creates a fully self-contained, project-native differential-drive robot named
Localbot that eliminates ALL dependencies on external Fuel/internet model hosting.

### Why Localbot?

The MovAI TugBot was loaded from fuel.ignitionrobotics.org (or Fuel cache) via
an HTTPS URI in the world SDF. This caused three compounding problems:

1. URDF↔SDF physics mismatch:
   TugBot wheel_radius=0.195m, wheel_separation=0.5605m
   URDF defined: wheel_radius=0.1m, wheel_separation=0.45m
   → Nav2 kinematics and odometry computations were based on wrong values

2. Joint name mismatch:
   TugBot SDF: wheel_left_joint / wheel_right_joint
   URDF expected: left_wheel_joint / right_wheel_joint
   → joint_state_relay needed complex name mapping at 50Hz

3. Unused plugins generating warnings and wasting CPU:
   Gripper JointControllers, LinearBatteryPlugin, PosePublisher,
   warnign_light_joint spinning at 10 rad/s (previously fixed to 'fixed'
   type but that only worked once Fuel URI was replaced with model://)

### What Localbot provides

- Zero Fuel/internet dependency: fully local, zero external URL references
- Exact URDF match: wheel_radius=0.1m, wheel_separation=0.45m (same as URDF)
- Exact joint name match: left_wheel_joint / right_wheel_joint (same as URDF)
  → joint_state_relay simplified to QoS-bridge-only (no name remapping)
- Only used sensors: RGB camera + depth_camera + IMU (no gripper, no lidar)
- Camera position matches URDF exactly: (0.0553, 0, 0.4323) from base_link
- optical_frame_id=camera_link_optical in sensors: matches URDF TF tree directly
  → tugbot/camera_front/color alias link in URDF removed (no longer needed)
- Simple geometry: box chassis + cylinder wheels + sphere casters
  → zero external mesh dependencies

### Files created

  src/ugv_sim/models/localbot/model.config  — Gazebo model discovery file
  src/ugv_sim/models/localbot/model.sdf     — Complete robot (800+ commented lines)

### Files modified

  src/ugv_sim/worlds/tugbot_warehouse.sdf
    - Replace <uri>model://tugbot</uri> with <uri>model://localbot</uri>
    - Update Teleop GUI plugin topic: /model/tugbot/cmd_vel → /model/localbot/cmd_vel
    - Spawn z reduced: 0.1 → 0.01 (correct ground clearance for Localbot wheel radius)

  src/ugv_sim/config/gazebo_bridge.yaml
    - All GZ topic paths updated: model/tugbot → model/localbot
    - Camera link name: camera_front → camera_link (matches Localbot SDF structure)
    - Extensive comments added (QoS rules, naming conventions, depth_image warning)

  src/ugv_sim/scripts/joint_state_relay.py
    - Simplified: no name mapping needed (Localbot names match URDF directly)
    - Now pure QoS bridge: BestEffort (GZ bridge) → Reliable (RSP)
    - Kept joint filter for safety (unknown joints still dropped silently)
    - Extensive documentation added explaining the design rationale

  src/ugv_description/urdf/ugv_base.urdf.xacro
    - Replaced tugbot_simp.dae mesh with navy-blue box (0.6×0.4×0.2m)
    - Added camera mast visual (matches Gazebo appearance)
    - Replaced wheel.dae mesh with orange cylinder (matches Localbot SDF)
    - Zero external mesh dependencies remaining in URDF

  src/ugv_description/urdf/sensors/camera.urdf.xacro
    - Removed tugbot/camera_front/color alias link and joint
    - Localbot sensor uses optical_frame_id=camera_link_optical directly
    - Added documentation explaining optical frame convention and position

  README.md
    - Complete modular rewrite: 20 sections, per-module documentation
    - Module Map diagram showing input/output topics for each component
    - Localbot documentation: spawning in custom worlds, GZ_SIM_RESOURCE_PATH
    - 'How to safely modify each module' section for independent development
    - All change history entries updated with current fixes

## Modular Project Structure

README now documents the project as independent modules:
  Simulation (ugv_sim)        — robot + world + bridge
  Robot Description (ugv_description) — URDF + TF
  Perception (ugv_perception) — depth relay + YOLO + point cloud
  SLAM (localization.launch)  — RTAB-Map 2D visual SLAM
  Navigation (navigation.launch) — Nav2: planner + controller + costmaps
  Terrain Analysis (ugv_terrain) — 2.5D traversability mapping

Each module section documents: what it provides, what it requires, all files,
key parameters with rationale, and how to safely modify it independently.

File: src/ugv_description/urdf/sensors/camera.urdf.xacro (robot description, xacro)
@@ -1,7 +1,25 @@
 <?xml version="1.0"?>
+<!--
+  camera.urdf.xacro — Camera link and optical frame definitions for Localbot.
+  Defines three links and their joints:
+    camera_link         : Physical camera housing (box geometry)
+    camera_link_optical : Standard ROS optical frame (Z-forward, X-right, Y-down)
+  The camera_link_optical frame is what Gazebo sensors publish image data in.
+  This must match the optical_frame_id set in Localbot's model.sdf sensor config.
+  Camera position (base_camera_joint) matches Localbot model.sdf camera_link pose:
+    camera_link in model frame = 0.0553 0 0.6323
+    = base_link(0 0 0.2) + base_camera_joint(0.0553 0 0.4323)
+  NOTE: The "tugbot/camera_front/color" alias link has been REMOVED.
+  The TugBot Fuel model published camera_info with frame_id "tugbot/camera_front/color",
+  requiring an alias TF link. Localbot's sensors use optical_frame_id="camera_link_optical"
+  directly, so no alias is needed. The TF tree is simpler and fully standard.
+-->
 <robot xmlns:xacro="http://www.ros.org/wiki/xacro">
-    <xacro:property name="camera_length" value="0.03" />
-    <xacro:property name="camera_width" value="0.10" />
-    <xacro:property name="camera_height" value="0.03" />
+    <!-- Camera housing dimensions -->
+    <xacro:property name="camera_length" value="0.03" />   <!-- depth (X) -->
+    <xacro:property name="camera_width"  value="0.10" />   <!-- width (Y) -->
+    <xacro:property name="camera_height" value="0.03" />   <!-- height (Z) -->
+    <!-- camera_link: physical camera housing mounted on Localbot's camera mast.
+         Visualized as a small dark-grey box in RViz. -->
     <link name="camera_link">
         <visual>
@@ -24,5 +42,9 @@
         </inertial>
     </link>
-    <!-- Tugbot camera_front link matching Gazebo SDF pose (0.0553, 0, 0.4323) -->
+    <!-- base_camera_joint: mount camera_link onto base_link at Localbot mast top.
+         Position matches Localbot model.sdf camera_link pose relative to base_link:
+           xyz = 0.0553 0 0.4323
+         (In model frame: 0.0553 0 0.2+0.4323=0.6323 — camera is 63cm from ground)
+         This joint is FIXED — camera does not move relative to chassis. -->
     <joint name="base_camera_joint" type="fixed">
         <parent link="base_link" />
@@ -30,5 +52,17 @@
         <origin xyz="0.0553 0 0.4323" rpy="0 0 0" />
     </joint>
-    <!-- Standard ROS optical frame convention -->
+    <!-- camera_link_optical: standard ROS camera optical frame.
+         Convention: Z-forward (into scene), X-right, Y-down.
+         This is the frame_id used for:
+           - /camera/image_raw     header.frame_id
+           - /camera/camera_info   header.frame_id
+           - /camera/depth/*       header.frame_id
+           - /perception/depth/*   header.frame_id (relayed)
+           - Nav2 ObstacleLayer    sensor_frame (inferred from point cloud)
+         Rotation rpy="-pi/2 0 -pi/2" converts from camera body frame to optical frame:
+           camera body: X-forward, Y-left, Z-up
+           optical:     X-right,   Y-down, Z-forward
+         Offset xyz="0 0.0325 0.0125" matches the color module position in Localbot SDF
+         (sensor pose <0 0.0325 0.0125> relative to camera_link). -->
     <link name="camera_link_optical" />
     <joint name="camera_optical_joint" type="fixed">
@@ -37,37 +71,3 @@
         <child link="camera_link_optical" />
     </joint>
-    <!-- Alias for Gazebo Tugbot frame_id: tugbot/camera_front/color -->
-    <link name="tugbot/camera_front/color" />
-    <joint name="tugbot_camera_color_joint" type="fixed">
-        <origin xyz="0 0 0" rpy="0 0 0" />
-        <parent link="camera_link_optical" />
-        <child link="tugbot/camera_front/color" />
-    </joint>
-    <gazebo reference="camera_link">
-        <sensor name="camera" type="camera">
-            <camera>
-                <horizontal_fov>1.3962634</horizontal_fov>
-                <image>
-                    <width>640</width>
-                    <height>480</height>
-                    <format>R8G8B8</format>
-                </image>
-                <clip>
-                    <near>0.1</near>
-                    <far>25.0</far>
-                </clip>
-                <noise>
-                    <type>gaussian</type>
-                    <mean>0.0</mean>
-                    <stddev>0.005</stddev>
-                </noise>
-                <optical_frame_id>camera_link_optical</optical_frame_id>
-                <camera_info_topic>camera/camera_info</camera_info_topic>
-            </camera>
-            <always_on>1</always_on>
-            <update_rate>30</update_rate>
-            <visualize>true</visualize>
-            <topic>camera/image_raw</topic>
-        </sensor>
-    </gazebo>
 </robot>

File: src/ugv_description/urdf/ugv_base.urdf.xacro (robot description, xacro)
@@ -10,9 +10,26 @@
     <link name="base_footprint" />
     <link name="base_link">
+        <!-- Localbot chassis: 0.6 × 0.4 × 0.2 m navy-blue box.
+             Matches Localbot model.sdf base_link visual exactly.
+             No external mesh dependency — box geometry is self-contained. -->
         <visual>
             <origin xyz="0 0 0" rpy="0 0 0" />
             <geometry>
-                <mesh filename="package://ugv_description/meshes/base/tugbot_simp.dae" />
+                <box size="${base_length} ${base_width} ${base_height}" />
             </geometry>
+            <material name="navy_blue">
+                <color rgba="0.1 0.1 0.7 1.0" />
+            </material>
+        </visual>
+        <!-- Camera mast visual: thin pole connecting chassis top to camera_link.
+             Purely decorative — makes RViz match Gazebo appearance. -->
+        <visual>
+            <origin xyz="0.0553 0 0.215" rpy="0 0 0" />
+            <geometry>
+                <box size="0.04 0.04 0.43" />
+            </geometry>
+            <material name="dark_grey">
+                <color rgba="0.3 0.3 0.3 1.0" />
+            </material>
         </visual>
         <collision>
@@ -37,9 +54,14 @@
     <xacro:macro name="wheel" params="prefix y_offset">
         <link name="${prefix}_wheel_link">
+            <!-- Orange cylinder wheel — matches Localbot SDF wheel visual.
+                 rpy rotates cylinder from default Z-axis to Y-axis (wheel axle direction). -->
             <visual>
-                <origin xyz="0 0 0" rpy="0 0 0" />
+                <origin xyz="0 0 0" rpy="${pi/2} 0 0" />
                 <geometry>
-                    <mesh filename="package://ugv_description/meshes/wheel/wheel.dae" />
+                    <cylinder radius="${wheel_radius}" length="${wheel_length}" />
                 </geometry>
+                <material name="orange">
+                    <color rgba="0.9 0.5 0.1 1.0" />
+                </material>
             </visual>
             <collision>
