Commit message: feat(ugv): YOLO26 upgrade, perception/terrain modularization, bugfixes & README overhaul
- Upgrade YOLO to YOLO26n-seg (NMS-free, FP16) with configurable hazard classes in perception.yaml
- Replace hardcoded perception launch dicts with centralized perception.yaml
- Vectorize terrain_analysis_node with TF2 camera transform, slope tolerance, and terrain.yaml
- Fix URDF wheel visual orientation mismatch (removed erroneous pi/2 roll)
- Fix model.sdf base_link ixx inertia calculation (0.2708 -> 0.2500)
- Modernize Gazebo Harmonic diff-drive & joint-state system plugin namespaces (gz-sim)
- Clean up dead code: unused hazard_mask_node, orphaned grid_map_* configs, outdated YAMLs
- Add missing runtime dependencies across ugv_bringup and ugv_sim package.xml files
- Register atexit cleanup hook for dynamic bridge tempfiles in sim.launch.py
- Complete README overhaul documenting pure-vision outdoor UGV architecture and YOLO26

File: src/ugv_description/urdf/ugv_base.urdf.xacro (robot description, xacro)
@@ -57,5 +57,5 @@
                  rpy rotates cylinder from default Z-axis to Y-axis (wheel axle direction). -->
             <visual>
-                <origin xyz="0 0 0" rpy="${pi/2} 0 0" />
+                <origin xyz="0 0 0" rpy="0 0 0" />
                 <geometry>
                     <cylinder radius="${wheel_radius}" length="${wheel_length}" />
